Commit message: updated naming scheme

File: src/kenny_description/urdf/camera_mechanism/camera_mechanism.urdf.xacro (robot description, xacro)
@@ -30,5 +30,5 @@
       </inertial>
     </link>
-    <joint name="joint_camera_pan_to_arm1" type="revolute">
+    <joint name="joint_camera_z_rotation" type="revolute">
       <!-- <parent link="arm_link1"/> -->
       <parent link="${parent}"/>
@@ -39,4 +39,5 @@
       <limit effort="1000.0" lower="${-pi/4}" upper="${pi/4}" velocity="0.5"/>
     </joint>
+    <!-- Link created for aesthetics (prevent floating y-rotation link) -->
     <link name="camera_tilt_block">
       <visual>
@@ -64,4 +65,5 @@
       <origin xyz="0 ${camera_pan_rad} ${camera_pan_rad-camera_tilt_block_width/2}" rpy="0 0 0"/>
     </joint>
+    <!-- Link/Joint responsible for tilting (rotating about y axis) -->
     <link name="camera_tilt_holder">
       <visual>
@@ -78,5 +80,5 @@
       </inertial>
     </link>
-    <joint name="joint_camera_tilt_block_to_holder" type="revolute">
+    <joint name="joint_camera_y_rotation" type="revolute">
       <parent link="camera_tilt_block"/>
       <child link="camera_tilt_holder"/>
@@ -85,6 +87,7 @@
       <limit effort="1000.0" lower="${-1*pi/6}" upper="${pi/6}" velocity="0.5"/>
     </joint>
-    <xacro:camera_joint name="camera_pan_to_arm1"/>
-    <xacro:camera_joint name="camera_tilt_block_to_holder"/>
+    <!-- call macros for defining transmission of camera joints -->
+    <xacro:camera_joint name="camera_z_rotation"/>
+    <xacro:camera_joint name="camera_y_rotation"/>
   </xacro:macro>
 </robot>
