Commit message: updated gazebo model

File: src/kenny_description/urdf/arm/arm.transmission.xacro (robot description, xacro)
@@ -2,5 +2,5 @@
 <robot xmlns:xacro="http://www.ros.org/wiki/xacro" name="kenny">
   <!-- Arm joint -->
-  <xacro:macro name="kenny_arm_joint" params="name">
+  <xacro:macro name="kenny_arm_joint_transmission" params="name">
     <transmission name="tran_${name}">
       <type>transmission_interface/SimpleTransmission</type>

File: src/kenny_description/urdf/arm/arm.urdf.xacro (robot description, xacro)
@@ -2,4 +2,6 @@
 <robot xmlns:xacro="http://www.ros.org/wiki/xacro">
   <xacro:include filename="$(find kenny_description)/urdf/arm/arm.transmission.xacro"/>
+  <xacro:include filename="$(find kenny_description)/urdf/arm/arm.gazebo.urdf"/>
+  <!--  ++++++++++++++++++++++++++++++++++++++++ -->
   <xacro:property name="link1_length" value="0.73"/>
   <xacro:property name="link1_width" value="0.378"/>
@@ -12,4 +14,5 @@
   <xacro:property name="link3_width" value="0.06"/>
   <xacro:property name="link3_depth" value="0.08"/>
+  <!--  ++++++++++++++++++++++++++++++++++++++++ -->
   <xacro:macro name="kenny_arm" params="parent *origin">
     <link name="reel">
@@ -60,8 +63,10 @@
       </inertial>
     </link>
-    <joint name="joint_reel_link1" type="fixed">
+    <joint name="joint_reel_link1" type="revolute">
         <parent link="reel"/>
         <child link="arm_link1"/>
         <origin xyz="${-1*reel_base_offset} 0 ${reel_length/2+link1_depth/2}" rpy="0 0 0"/>
+        <axis xyz="0 1 0"/>
+        <limit effort="1000.0" lower="0" upper="0" velocity="0"/>
     </joint>
     <link name="arm_link2">
@@ -121,7 +126,9 @@
     </joint>
     <!-- Transmission Macros -->
-    <xacro:kenny_arm_joint name="link1_link2"/>
-    <xacro:kenny_arm_joint name="link2_link3"/>
-    <xacro:kenny_arm_joint name="reel_link1"/>
+    <xacro:kenny_arm_joint_transmission name="reel_link1"/>
+    <xacro:kenny_arm_joint_transmission name="link1_link2"/>
+    <xacro:kenny_arm_joint_transmission name="link2_link3"/>
+    <!-- Gazebo Macro -->
+    <xacro:arm_gazebo/>
   </xacro:macro>
 </robot>

File: src/kenny_description/urdf/base/base.urdf.xacro (robot description, xacro)
@@ -1,4 +1,7 @@
 <?xml version="1.0"?>
 <robot xmlns:xacro="http://www.ros.org/wiki/xacro">
+  <!-- <xacro:include filename="$(find kenny_description)/urdf/base/base.transmission.xacro"/> -->
+  <xacro:include filename="$(find kenny_description)/urdf/base/base.gazebo.urdf"/>
+  <!--  ++++++++++++++++++++++++++++++++++++++++ -->
   <xacro:property name="base_length" value="1.176" />
   <xacro:property name="base_width" value="0.444" />
@@ -11,4 +14,5 @@
   <xacro:property name="reel_length" value="0.09" />
   <xacro:property name="reel_base_offset" value="0.0" />
+  <!--  ++++++++++++++++++++++++++++++++++++++++ -->
   <xacro:macro name="wheel" params="name reflect">
     <link name="${name}">
@@ -62,4 +66,5 @@
     <xacro:wheel name="wheel_right" reflect="1" />
     <xacro:wheel name="wheel_left" reflect="-1"/>
+    <xacro:base_gazebo/>
   </xacro:macro>
 </robot>

File: src/kenny_description/urdf/camera_mechanism/camera_mechanism.urdf.xacro (robot description, xacro)
@@ -2,4 +2,6 @@
 <robot xmlns:xacro="http://www.ros.org/wiki/xacro">
   <xacro:include filename="$(find kenny_description)/urdf/camera_mechanism/camera_mechanism.transmission.urdf"/>
+  <xacro:include filename="$(find kenny_description)/urdf/camera_mechanism/camera_mechanism.gazebo.urdf"/>
+  <!--  ++++++++++++++++++++++++++++++++++++++++ -->
   <xacro:property name="camera_pan_rad" value="0.095"/>
   <xacro:property name="camera_pan_length" value="0.023"/>
@@ -10,4 +12,5 @@
   <xacro:property name="camera_tilt_holder_width" value="0.153"/>
   <xacro:property name="camera_tilt_holder_depth" value="0.102"/>
+  <!--  ++++++++++++++++++++++++++++++++++++++++ -->
   <xacro:macro name="camera_mechanism" params="parent *origin">
     <link name="camera_pan">
@@ -90,4 +93,5 @@
     <xacro:camera_joint name="camera_z_rotation"/>
     <xacro:camera_joint name="camera_y_rotation"/>
+    <xacro:camera_mechanism_gazebo/>
   </xacro:macro>
 </robot>

Commit message: moveit compatibility edits

File: src/kenny_description/urdf/arm/arm.transmission.xacro (robot description, xacro)
@@ -1,4 +1,4 @@
 <?xml version="1.0"?>
-<robot xmlns:xacro="http://www.ros.org/wiki/xacro" name="kenny">
+<robot xmlns:xacro="http://www.ros.org/wiki/xacro" name="kenny_arm">
   <!-- Arm joint -->
   <xacro:macro name="kenny_arm_joint_transmission" params="name">

File: src/kenny_description/urdf/arm/arm.urdf.xacro (robot description, xacro)
@@ -1,4 +1,5 @@
 <?xml version="1.0"?>
-<robot xmlns:xacro="http://www.ros.org/wiki/xacro">
+<robot xmlns:xacro="http://www.ros.org/wiki/xacro" name="kenny_arm">
+<!-- <robot xmlns:xacro="http://www.ros.org/wiki/xacro"> -->
   <xacro:include filename="$(find kenny_description)/urdf/arm/arm.transmission.xacro"/>
   <xacro:include filename="$(find kenny_description)/urdf/arm/arm.gazebo.urdf"/>
@@ -18,5 +19,5 @@
   <xacro:property name="reel_base_offset" value="0.0" />
   <!--  ++++++++++++++++++++++++++++++++++++++++ -->
-  <xacro:macro name="kenny_arm" params="parent *origin">
+  <xacro:macro name="kenny_arm" > <!-- params="parent *origin"> -->
     <link name="reel">
       <visual>
@@ -41,5 +42,5 @@
     <!-- fixed joints do not exist in gazebo models (SDF file format),
          fixed joint is now revolute with 0 degrees of motion -->
-    <joint name="joint_base_reel" type="revolute">
+    <!-- <joint name="joint_base_reel" type="revolute">
       <parent link="${parent}"/>
       <child link="reel"/>
@@ -47,5 +48,5 @@
       <xacro:insert_block name="origin" />
         <limit effort="1000.0" lower="0" upper="0" velocity="0"/>
-    </joint>
+    </joint> -->
     <link name="arm_link1">
       <visual>
@@ -67,5 +68,5 @@
       </inertial>
     </link>
-    <joint name="joint_base_link1" type="continuous">
+    <joint name="joint_reel_link1" type="continuous">
         <parent link="reel"/>
         <child link="arm_link1"/>
@@ -134,5 +135,5 @@
     <xacro:kenny_arm_joint_transmission name="link2_link3"/>
     <!-- Gazebo Macro -->
-    <xacro:arm_gazebo/>
+    <xacro:kenny_arm_gazebo/>
   </xacro:macro>
 </robot>

File: src/kenny_description/urdf/kenny.urdf (robot description, URDF)
Before this commit: robot kenny, 0 links, 0 joints
Joints:
- added joint arm_mount_joint: type fixed, parent base_link, child reel, origin xyz=${reel_base_offset} 0 ${base_depth+off_floor+0.5*reel_length}
