Commit message: successfully split into sep dirs

File: src/kenny_description/urdf/arm/arm.urdf.xacro (robot description, xacro)
@@ -28,5 +28,5 @@
     </link>
     <joint name="base_to_reel" type="continuous">
-      <parent link="$(parent)"/>
+      <parent link="${parent}"/>
       <child link="reel"/>
       <axis xyz="0 0 1"/>

File: src/kenny_description/urdf/base/base.urdf.xacro (robot description, xacro)
@@ -4,5 +4,5 @@
   <xacro:property name="base_width" value="0.444" />
   <xacro:property name="base_depth" value="0.308" />
-  <xacro:property name="off_floor" value="0.1" />
+  <xacro:property name="off_floor" value="0.05" />
   <xacro:property name="wheel_length" value="1.135" />
   <xacro:property name="wheel_width" value="0.12" />
@@ -11,11 +11,11 @@
   <xacro:property name="reel_length" value="0.09" />
   <xacro:property name="reel_base_offset" value="0.0" />
-  <xacro:macro name="kenny_base" params="name">
-    <link name="$(name)_link">
+  <xacro:macro name="kenny_base" >
+    <link name="base_link">
       <visual>
         <geometry>
             <box size="${base_length} ${base_width} ${base_depth}"/>
         </geometry>
-        <origin xyz="0 0 ${off_floor}" />
+        <origin xyz="0 0 ${off_floor+base_depth/2}" />
         <material name="yellow"/>
       </visual>
@@ -24,29 +24,6 @@
             <box size="${base_length} ${base_width} ${base_depth}"/>
         </geometry>
-        <origin xyz="0 0 ${off_floor+base_depth/2}" />
-    </collision>
-    </link>
-    <!-- base_footprint is a fictitious link(frame) that is on the ground right below base_link origin,
-    navigation stack dedpends on this frame -->
-    <link name="${name}_footprint">
-      <inertial>
-        <mass value="1.0" />
+        <!-- <origin xyz="0 0 ${off_floor+base_depth/2}" /> -->
         <origin xyz="0 0 0" />
-        <inertia ixx="0.01" ixy="0.0" ixz="0.0"
-                iyy="0.01" iyz="0.0" izz="0.01" />
-      </inertial>
-      <visual>
-        <origin xyz="0 0 0" rpy="0 0 0" />
-        <geometry>
-          <box size="0.01 0.01 0.01" />
-        </geometry>
-        <material name="White" />
-      </visual>
-      <collision>
-        <!-- represent base collision with a simple rectangular model -->
-        <origin xyz="0 0 0.05" rpy="0 0 0" />
-        <geometry>
-          <box size="0.001 0.001 0.001" />
-        </geometry>
       </collision>
     </link>

File: src/kenny_description/urdf/kenny.urdf (robot description, URDF)
Before this commit: robot kenny, 3 links, 3 joints
Links:
- removed link camera_pan
- removed link camera_tilt_block
- removed link camera_tilt_holder
Joints:
- removed joint camera_pan_to_arm1
- removed joint camera_tilt_block_to_holder
- removed joint camera_tilt_block_to_pan

File: src/kenny_description/urdf/materials.urdf.xacro (robot description, xacro)
@@ -1,4 +1,4 @@
 <?xml version="1.0"?>
-<<robot>
+<robot>
     <material name="yellow">
         <color rgba="0.98 0.85 0.37 1"/>

Commit message: issue: controller manager not launching

File: src/kenny_description/urdf/arm/arm.urdf.xacro (robot description, xacro)
@@ -1,4 +1,5 @@
 <?xml version="1.0"?>
 <robot xmlns:xacro="http://www.ros.org/wiki/xacro">
+  <xacro:include filename="$(find kenny_description)/urdf/arm/arm.transmission.xacro"/>
   <xacro:property name="link1_length" value="0.73"/>
   <xacro:property name="link1_width" value="0.378"/>
@@ -26,4 +27,9 @@
           <!-- <origin xyz="0 0 0"/> -->
         </collision>
+      <inertial>
+        <origin xyz="0 0 0" rpy="0 0 0"/>
+        <mass value="1"/>
+        <inertia ixx="0.2" ixy="0.0" ixz="0.0" iyy="0.2" iyz="0.0" izz="0.2"/>
+      </inertial>
     </link>
     <joint name="base_to_reel" type="continuous">
@@ -36,18 +42,23 @@
     </joint>
     <link name="arm_link1">
-        <visual>
-          <geometry>
-            <box size="${link1_length} ${link1_width} ${link1_depth}"/>
-          </geometry>
-          <material name="yellow"/>
-          <origin xyz="0 0 0" rpy="0 0 0"/>
-        </visual>
-        <collision>
-          <geometry>
-            <box size="${link1_length} ${link1_width} ${link1_depth}"/>
-          </geometry>
-        </collision>
+      <visual>
+        <geometry>
+          <box size="${link1_length} ${link1_width} ${link1_depth}"/>
+        </geometry>
+        <material name="yellow"/>
+        <origin xyz="0 0 0" rpy="0 0 0"/>
+      </visual>
+      <collision>
+        <geometry>
+          <box size="${link1_length} ${link1_width} ${link1_depth}"/>
+        </geometry>
+      </collision>
+      <inertial>
+        <origin xyz="0 0 0" rpy="0 0 0"/>
+        <mass value="1"/>
+        <inertia ixx="0.2" ixy="0.0" ixz="0.0" iyy="0.2" iyz="0.0" izz="0.2"/>
+      </inertial>
     </link>
-    <joint name="reel_to_link1" type="fixed">
+    <joint name="joint_reel_link1" type="fixed">
         <parent link="reel"/>
         <child link="arm_link1"/>
@@ -68,6 +79,11 @@
         <origin xyz="0 0 ${link2_length/2}" rpy="0 0 0"/>
       </collision>
+      <inertial>
+        <origin xyz="0 0 0" rpy="0 0 0"/>
+        <mass value="1"/>
+        <inertia ixx="0.2" ixy="0.0" ixz="0.0" iyy="0.2" iyz="0.0" izz="0.2"/>
+      </inertial>
     </link>
-    <joint name="link1_to_link2" type="revolute">
+    <joint name="joint_link1_link2" type="revolute">
       <parent link="arm_link1"/>
       <child link="arm_link2"/>
@@ -91,12 +107,21 @@
         <origin xyz="${link3_length/2} 0 0" rpy="0 0 0"/>
       </collision>
+      <inertial>
+        <origin xyz="0 0 0" rpy="0 0 0"/>
+        <mass value="1"/>
+        <inertia ixx="0.2" ixy="0.0" ixz="0.0" iyy="0.2" iyz="0.0" izz="0.2"/>
+      </inertial>
     </link>
-    <joint name="link2_to_link3" type="revolute">
+    <joint name="joint_link2_link3" type="revolute">
       <parent link="arm_link2"/>
       <child link="arm_link3"/>
       <axis xyz="0 1 0"/>
-      <origin xyz="0 0 ${link2_length}" rpy="0 0.84 0"/>
-      <limit effort="1000.0" lower="-0.84" upper="0" velocity="0.5"/>
+      <origin xyz="0 0 ${link2_length}" rpy="0 0 0"/>
+      <limit effort="1000.0" lower="0" upper="0.84" velocity="0.5"/>
     </joint>
+    <!-- Transmission Macros -->
+    <xacro:kenny_arm_joint name="link1_link2"/>
+    <xacro:kenny_arm_joint name="link2_link3"/>
+    <xacro:kenny_arm_joint name="reel_link1"/>
   </xacro:macro>
 </robot>

File: src/kenny_description/urdf/base/base.urdf.xacro (robot description, xacro)
@@ -11,4 +11,31 @@
   <xacro:property name="reel_length" value="0.09" />
   <xacro:property name="reel_base_offset" value="0.0" />
+  <xacro:macro name="wheel" params="name reflect">
+    <link name="${name}">
+      <visual>
+        <geometry>
+          <box size="${wheel_length} ${wheel_width} ${wheel_depth}"/>
+        </geometry>
+        <origin xyz="0 0 0"/>
+        <material name="black"/>
+      </visual>
+      <collision>
+        <geometry>
+            <box size="${wheel_length} ${wheel_width} ${wheel_depth}"/>
+        </geometry>
+        <!-- <origin xyz="0 0 0"/> -->
+      </collision>
+      <inertial>
+        <origin xyz="0 0 ${+0.5*base_depth}" rpy="0 0 0"/>
+        <mass value="1"/>
+        <inertia ixx="0.2" ixy="0.0" ixz="0.0" iyy="0.2" iyz="0.0" izz="0.2"/>
+      </inertial>
+    </link>
+    <joint name="base_to_${name}" type="fixed">
+      <parent link="base_link"/>
+      <child link="${name}"/>
+      <origin xyz="0 ${reflect * 0.5*(base_width+wheel_width)} ${-off_floor+wheel_depth/2}" />
+    </joint>
+  </xacro:macro>
   <xacro:macro name="kenny_base" >
     <link name="base_link">
@@ -27,45 +54,12 @@
         <origin xyz="0 0 0" />
       </collision>
+      <inertial>
+        <origin xyz="0 0 ${off_floor+0.5*base_depth}" rpy="0 0 0"/>
+        <mass value="1"/>
+        <inertia ixx="0.2" ixy="0.0" ixz="0.0" iyy="0.2" iyz="0.0" izz="0.2"/>
+      </inertial>
     </link>
-    <link name="wheel_left">
-      <visual>
-        <geometry>
-          <box size="${wheel_length} ${wheel_width} ${wheel_depth}"/>
-        </geometry>
-        <origin xyz="0 0 0"/>
-        <material name="black"/>
-      </visual>
-      <collision>
-        <geometry>
-          <box size="${wheel_length} ${wheel_width} ${wheel_depth}"/>
-        </geometry>
-        <!-- <origin xyz="0 0 0"/> -->
-      </collision>
-    </link>
-    <joint name="base_to_wheel_left" type="fixed">
-      <parent link="base_link"/>
-      <child link="wheel_left"/>
-      <origin xyz="0 ${-0.5*(base_width+wheel_width)} ${-off_floor+wheel_depth/2}" />
-    </joint>
-    <link name="wheel_right">
-      <visual>
-        <geometry>
-          <box size="${wheel_length} ${wheel_width} ${wheel_depth}"/>
-        </geometry>
-        <origin xyz="0 0 0"/>
-        <material name="black"/>
-      </visual>
-      <collision>
-        <geometry>
-            <box size="${wheel_length} ${wheel_width} ${wheel_depth}"/>
-        </geometry>
-        <!-- <origin xyz="0 0 0"/> -->
-      </collision>
-    </link>
-    <joint name="base_to_wheel_right" type="fixed">
-      <parent link="base_link"/>
-      <child link="wheel_right"/>
-      <origin xyz="0 ${0.5*(base_width+wheel_width)} ${-off_floor+wheel_depth/2}" />
-    </joint>
+    <xacro:wheel name="wheel_right" reflect="1" />
+    <xacro:wheel name="wheel_left" reflect="-1"/>
   </xacro:macro>
 </robot>

File: src/kenny_description/urdf/camera_mechanism/camera_mechanism.urdf.xacro (robot description, xacro)
@@ -1,4 +1,5 @@
 <?xml version="1.0"?>
 <robot xmlns:xacro="http://www.ros.org/wiki/xacro">
+  <xacro:include filename="$(find kenny_description)/urdf/camera_mechanism/camera_mechanism.transmission.urdf"/>
   <xacro:property name="camera_pan_rad" value="0.095"/>
   <xacro:property name="camera_pan_length" value="0.023"/>
@@ -23,6 +24,11 @@
         </geometry>
       </collision>
+      <inertial>
+        <origin xyz="0 0 0" rpy="0 0 0"/>
+        <mass value="1"/>
+        <inertia ixx="0.2" ixy="0.0" ixz="0.0" iyy="0.2" iyz="0.0" izz="0.2"/>
+      </inertial>
     </link>
-    <joint name="camera_pan_to_arm1" type="revolute">
+    <joint name="joint_camera_pan_to_arm1" type="revolute">
       <!-- <parent link="arm_link1"/> -->
       <parent link="${parent}"/>
@@ -46,4 +52,9 @@
         </geometry>
       </collision>
+      <inertial>
+        <origin xyz="0 0 0" rpy="0 0 0"/>
+        <mass value="1"/>
+        <inertia ixx="0.2" ixy="0.0" ixz="0.0" iyy="0.2" iyz="0.0" izz="0.2"/>
+      </inertial>
     </link>
     <joint name="camera_tilt_block_to_pan" type="fixed">
@@ -61,6 +72,11 @@
         <material name="yellow"/>
       </visual>
+      <inertial>
+        <origin xyz="0 0 0" rpy="0 0 0"/>
+        <mass value="1"/>
+        <inertia ixx="0.2" ixy="0.0" ixz="0.0" iyy="0.2" iyz="0.0" izz="0.2"/>
+      </inertial>
     </link>
-    <joint name="camera_tilt_block_to_holder" type="revolute">
+    <joint name="joint_camera_tilt_block_to_holder" type="revolute">
       <parent link="camera_tilt_block"/>
       <child link="camera_tilt_holder"/>
@@ -69,4 +85,6 @@
       <limit effort="1000.0" lower="${-1*pi/6}" upper="${pi/6}" velocity="0.5"/>
     </joint>
+    <xacro:camera_joint name="camera_pan_to_arm1"/>
+    <xacro:camera_joint name="camera_tilt_block_to_holder"/>
   </xacro:macro>
 </robot>

Commit message: added joint controllers

File: src/kenny_description/urdf/arm/arm.urdf.xacro (robot description, xacro)
@@ -14,4 +14,7 @@
   <xacro:property name="link3_width" value="0.06"/>
   <xacro:property name="link3_depth" value="0.08"/>
+  <xacro:property name="reel_rad" value="0.199" />
+  <xacro:property name="reel_length" value="0.09" />
+  <xacro:property name="reel_base_offset" value="0.0" />
   <!--  ++++++++++++++++++++++++++++++++++++++++ -->
   <xacro:macro name="kenny_arm" params="parent *origin">
@@ -36,9 +39,10 @@
       </inertial>
     </link>
-    <joint name="base_to_reel" type="continuous">
+    <joint name="base_to_reel" type="revolute">
       <parent link="${parent}"/>
       <child link="reel"/>
       <axis xyz="0 0 1"/>
       <xacro:insert_block name="origin" />
+        <limit effort="1000.0" lower="0" upper="0" velocity="0"/>
       <!-- <origin xyz="${reel_base_offset} 0 ${base_depth}" /> -->
       <!-- <origin xyz="${reel_base_offset} 0 0" /> -->
@@ -63,10 +67,10 @@
       </inertial>
     </link>
-    <joint name="joint_reel_link1" type="revolute">
+    <joint name="joint_base_link1" type="continuous">
         <parent link="reel"/>
         <child link="arm_link1"/>
         <origin xyz="${-1*reel_base_offset} 0 ${reel_length/2+link1_depth/2}" rpy="0 0 0"/>
-        <axis xyz="0 1 0"/>
-        <limit effort="1000.0" lower="0" upper="0" velocity="0"/>
+        <axis xyz="0 0 1"/>
+        <!-- <limit effort="1000.0" lower="0" upper="0" velocity="0"/> -->
     </joint>
     <link name="arm_link2">

File: src/kenny_description/urdf/base/base.urdf.xacro (robot description, xacro)
@@ -11,7 +11,4 @@
   <xacro:property name="wheel_width" value="0.12" />
   <xacro:property name="wheel_depth" value="0.338" />
-  <xacro:property name="reel_rad" value="0.199" />
-  <xacro:property name="reel_length" value="0.09" />
-  <xacro:property name="reel_base_offset" value="0.0" />
   <!--  ++++++++++++++++++++++++++++++++++++++++ -->
   <xacro:macro name="wheel" params="name reflect">

Commit message: cleaned and renamed joints

File: src/kenny_description/urdf/arm/arm.urdf.xacro (robot description, xacro)
@@ -27,10 +27,10 @@
         <material name="yellow"/>
       </visual>
-        <collision>
-          <geometry>
-              <cylinder length="${reel_length}" radius="${reel_rad}"/>
-          </geometry>
-          <!-- <origin xyz="0 0 0"/> -->
-        </collision>
+      <collision>
+        <geometry>
+            <cylinder length="${reel_length}" radius="${reel_rad}"/>
+        </geometry>
+        <!-- <origin xyz="0 0 0"/> -->
+      </collision>
       <inertial>
         <origin xyz="0 0 0" rpy="0 0 0"/>
@@ -39,5 +39,7 @@
       </inertial>
     </link>
-    <joint name="base_to_reel" type="revolute">
+    <!-- fixed joints do not exist in gazebo models (SDF file format),
+         fixed joint is now revolute with 0 degrees of motion -->
+    <joint name="joint_base_reel" type="revolute">
       <parent link="${parent}"/>
       <child link="reel"/>
@@ -45,6 +47,4 @@
       <xacro:insert_block name="origin" />
         <limit effort="1000.0" lower="0" upper="0" velocity="0"/>
-      <!-- <origin xyz="${reel_base_offset} 0 ${base_depth}" /> -->
-      <!-- <origin xyz="${reel_base_offset} 0 0" /> -->
     </joint>
     <link name="arm_link1">
@@ -130,5 +130,5 @@
     </joint>
     <!-- Transmission Macros -->
-    <xacro:kenny_arm_joint_transmission name="reel_link1"/>
+    <xacro:kenny_arm_joint_transmission name="base_link1"/>
     <xacro:kenny_arm_joint_transmission name="link1_link2"/>
     <xacro:kenny_arm_joint_transmission name="link2_link3"/>

Commit message: fixing parent of arm macro

File: src/kenny_description/urdf/arm/arm.urdf.xacro (robot description, xacro)
@@ -19,7 +19,8 @@
   <xacro:property name="reel_base_offset" value="0.0" />
   <!--  ++++++++++++++++++++++++++++++++++++++++ -->
-  <xacro:macro name="kenny_arm" params="parent"> <!-- params="parent *origin"> -->
+  <!-- <xacro:macro name="kenny_arm" params="parent"> params="parent *origin"> -->
+  <xacro:macro name="kenny_arm" params="parent *origin">
     <link name="dummy_reel">
-      <visual>
+      <!-- <visual>
         <geometry>
           <cylinder length="${reel_length/4}" radius="${reel_rad}"/>
@@ -27,6 +28,6 @@
         <origin xyz="0 0 0" rpy="0 0 0"/>
         <material name="yellow"/>
-      </visual>
-      <collision>
+      </visual> -->
+      <!-- <collision>
         <geometry>
             <cylinder length="${reel_length}" radius="${reel_rad}"/>
@@ -37,10 +38,12 @@
         <mass value="1"/>
         <inertia ixx="0" ixy="0.0" ixz="0.0" iyy="0.2" iyz="0.0" izz="0"/>
-      </inertial>
+      </inertial> -->
     </link>
     <joint name="dummy_reel_joint" type="revolute">
+      <!-- <parent link="base_link"/> -->
       <parent link="${parent}"/>
       <child link="dummy_reel"/>
-      <axis xyz="0 0 0"/>
+      <xacro:insert_block name="origin"/>
+      <axis xyz="0 0 1"/>
       <limit effort="1000.0" lower="0" upper="0" velocity="0"/>
     </joint>
@@ -70,6 +73,7 @@
       <child link="reel"/>
       <axis xyz="0 0 1"/>
+      <origin xyz="0 0 0" rpy="0 0 0"/>
       <!-- <xacro:insert_block name="origin" /> -->
-      <limit effort="1000.0" lower="0" upper="0" velocity="0"/>
+      <limit effort="1000.0" lower="-180" upper="180" velocity="2"/>
     </joint>
     <link name="arm">

File: src/kenny_description/urdf/base/base.urdf.xacro (robot description, xacro)
@@ -77,4 +77,6 @@
   <!--  ++++++++++++++++++++++++++++++++++++++++ -->
   <xacro:macro name="kenny_base" >
+  <!-- footprint link is used for calculating distances between
+        the robot and obstacles -->
     <link name="base_footprint">
       <origin xyz="0 0 0"/>
@@ -85,5 +87,4 @@
             <box size="${base_length} ${base_width} ${base_depth}"/>
         </geometry>
-        <!-- <origin xyz="0 0 ${off_floor+base_depth/2}" /> -->
         <origin xyz="0 0 0"/>
         <material name="yellow"/>
@@ -93,12 +94,11 @@
             <box size="${base_length} ${base_width} ${base_depth}"/>
         </geometry>
-        <!-- <origin xyz="0 0 ${off_floor+base_depth/2}" /> -->
         <origin xyz="0 0 0" />
       </collision>
     </link>
     <joint name="base_footprint_joint" type="fixed">
-      <parent link="base_link"/>
-      <child link="base_footprint"/>
-      <origin xyz="0 0 ${off_floor+base_depth/2}" />
+      <parent link="base_footprint"/>
+      <child link="base_link"/>
+      <origin xyz="0 0 ${off_floor}" />
     </joint>
     <link name="inertial_link">

File: src/kenny_description/urdf/kenny.urdf (robot description, URDF)
Before this commit: robot kenny, 0 links, 1 joints
Joints:
- removed joint arm_mount_joint

Commit message: trying to launch controllers

File: src/kenny_description/urdf/arm/arm.urdf.xacro (robot description, xacro)
@@ -96,10 +96,10 @@
     </link>
     <!-- link between reel and arm -->
-    <joint name="shoulder" type="revolute">
+    <joint name="shoulder" type="continuous">
         <parent link="dummy_reel"/>
         <child link="arm"/>
         <origin xyz="${-1*reel_base_offset} 0 ${reel_length/2+arm_depth/2}" rpy="0 0 0"/>
         <axis xyz="0 0 1"/>
-        <limit effort="1000.0" lower="-20" upper="20" velocity="0"/>
+        <limit effort="1000.0" velocity="0"/>
     </joint>
     <link name="forearm">

Commit message: base and arm controllers

File: src/kenny_description/urdf/arm/arm.urdf.xacro (robot description, xacro)
@@ -1,4 +1,4 @@
 <?xml version="1.0"?>
-<robot xmlns:xacro="http://www.ros.org/wiki/xacro" name="kenny_arm">
+<robot xmlns:xacro="http://www.ros.org/wiki/xacro" name="kenny">
 <!-- <robot xmlns:xacro="http://www.ros.org/wiki/xacro"> -->
   <xacro:include filename="$(find kenny_description)/urdf/arm/arm.transmission.xacro"/>
@@ -18,25 +18,6 @@
   <xacro:property name="reel_base_offset" value="0.0" />
   <!--  ++++++++++++++++++++++++++++++++++++++++ -->
-  <!-- <xacro:macro name="kenny_arm" params="parent"> params="parent *origin"> -->
   <xacro:macro name="kenny_arm" params="parent *origin">
-    <link name="dummy_reel">
-      <!-- <visual>
-        <geometry>
-          <cylinder length="${reel_length/4}" radius="${reel_rad}"/>
-        </geometry>
-        <origin xyz="0 0 0" rpy="0 0 0"/>
-        <material name="yellow"/>
-      </visual> -->
-      <!-- <collision>
-        <geometry>
-            <cylinder length="${reel_length}" radius="${reel_rad}"/>
-        </geometry>
-      </collision>
-      <inertial>
-        <origin xyz="0 0 0" rpy="0 0 0"/>
-        <mass value="1"/>
-        <inertia ixx="0" ixy="0.0" ixz="0.0" iyy="0.2" iyz="0.0" izz="0"/>
-      </inertial> -->
-    </link>
+    <link name="dummy_reel"/>
     <joint name="dummy_reel_joint" type="revolute">
       <!-- <parent link="base_link"/> -->
