Commit message: use xacro for parametric modelling

File: src/kenny_description/urdf/kenny.urdf (robot description, URDF)
Before this commit: robot kenny, 4 links, 3 joints
Links:
- removed link neck_base
- added link reel; visual cylinder length=${reel_length} radius=${reel_rad}
- link base_link: geometry visual box size=${base_length} ${base_width} ${base_depth}
- link wheel_left: geometry visual box size=${wheel_length} ${wheel_width} ${wheel_depth}
- link wheel_right: geometry visual box size=${wheel_length} ${wheel_width} ${wheel_depth}
Joints:
- removed joint base_to_neck
- added joint base_to_reel: type continuous, parent base_link, child reel, axis 0 0 1

Commit message: arm visuals (no joint movement)

File: src/kenny_description/urdf/kenny.urdf (robot description, URDF)
Before this commit: robot kenny, 4 links, 3 joints
Links:
- added link arm_link1; visual box size=${link1_length} ${link1_width} ${link1_depth}
- added link arm_link2; visual box size=${link2_depth} ${link2_width} ${link2_length}
- added link arm_link3; visual box size=${link3_length} ${link3_width} ${link3_depth}
Joints:
- added joint link1_to_link2: type fixed, parent arm_link1, child arm_link2
- added joint link2_to_link3: type fixed, parent arm_link2, child arm_link3
- added joint reel_to_link1: type fixed, parent reel, child arm_link1
- joint base_to_reel: axis 0 0 1 -> (none); type continuous -> fixed

Commit message: joints active, collisions started

File: src/kenny_description/urdf/kenny.urdf (robot description, URDF)
Before this commit: robot kenny, 7 links, 6 joints
Links:
- link arm_link1: geometry collision box size=${link1_length} ${link1_width} ${link1_depth}; visual box size=${link1_length} ${link1_width} ${link1_depth}
- link arm_link2: geometry collision box size=${link2_depth} ${link2_width} ${link2_length}; visual box size=${link2_depth} ${link2_width} ${link2_length}
- link arm_link3: geometry collision box size=${link3_length} ${link3_width} ${link3_depth}; visual box size=${link3_length} ${link3_width} ${link3_depth}
- link base_link: geometry collision box size=${base_length} ${base_width} ${base_depth}; visual box size=${base_length} ${base_width} ${base_depth}
- link reel: geometry collision cylinder length=${reel_length} radius=${reel_rad}; visual cylinder length=${reel_length} radius=${reel_rad}
- link wheel_left: geometry collision box size=${wheel_length} ${wheel_width} ${wheel_depth}; visual box size=${wheel_length} ${wheel_width} ${wheel_depth}
- link wheel_right: geometry collision box size=${wheel_length} ${wheel_width} ${wheel_depth}; visual box size=${wheel_length} ${wheel_width} ${wheel_depth}
Joints:
- joint base_to_reel: axis (none) -> 0 0 1; origin (none) -> xyz=${reel_base_offset} 0 ${base_depth+reel_length/2}; type fixed -> continuous
- joint base_to_wheel_left: origin (none) -> xyz=0 ${-0.5*(base_width+wheel_width)} ${off_floor+(off_floor - wheel_depth)/2}
- joint base_to_wheel_right: origin (none) -> xyz=0 ${0.5*(base_width+wheel_width)} ${off_floor+(off_floor - wheel_depth)/2}
- joint link1_to_link2: axis (none) -> 0 1 0; origin (none) -> xyz=${link1_length/2-link2_depth/2} 0 0 rpy=0 0 0; type fixed -> continuous
- joint link2_to_link3: axis (none) -> 0 1 0; origin (none) -> xyz=0 0 ${link2_length} rpy=0 0 0; type fixed -> continuous
- joint reel_to_link1: origin (none) -> xyz=${reel_base_offset/2} 0 ${reel_length/2+link1_depth/2} rpy=0 0 0

Commit message: arm moves according to physical limits of bot

File: src/kenny_description/urdf/kenny.urdf (robot description, URDF)
Before this commit: robot kenny, 7 links, 6 joints
Joints:
- joint link1_to_link2: limit (none) -> lower=0 upper=1.65 effort=1000.0 velocity=0.5; origin xyz=${link1_length/2-link2_depth/2} 0 0 rpy=0 0 0 -> xyz=${link1_length/2} 0 0 rpy=0 ${link2_default_rotation} 0; type continuous -> revolute
- joint link2_to_link3: limit (none) -> lower=-0.84 upper=0 effort=1000.0 velocity=0.5; origin xyz=0 0 ${link2_length} rpy=0 0 0 -> xyz=0 0 ${link2_length} rpy=0 0.84 0; type continuous -> revolute
- joint reel_to_link1: origin xyz=${reel_base_offset/2} 0 ${reel_length/2+link1_depth/2} rpy=0 0 0 -> xyz=${-1*reel_base_offset} 0 ${reel_length/2+link1_depth/2} rpy=0 0 0

Commit message: camera holder model, tilit link fails

File: src/kenny_description/urdf/kenny.urdf (robot description, URDF)
Before this commit: robot kenny, 7 links, 6 joints
Links:
- added link camera_pan; collision cylinder length=${camera_pan_length} radius=${camera_pan_rad}; visual cylinder length=${camera_pan_length} radius=${camera_pan_rad}
- added link camera_tilt; collision box size=${camera_tilt_length} ${camera_tilt_width} ${camera_tilt_de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; visual box size=${camera_tilt_length} ${camera_tilt_width} ${camera_tilt_de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
Joints:
- added joint camera_pan_to_arm1: type revolute, parent arm_link1, child camera_pan, origin xyz=${pan_arm_offset} 0 ${link1_depth/2} rpy=0 0 0, axis 0 0 1, limit lower=-0.84 upper=0 effort=1000.0 velocity=0.5
- added joint camera_tilt_to_pan: type revolute, origin xyz=0 0 ${camera_pan_length/2+camera_tilt_length} rpy=0 0 0, axis 0 1 0, limit lower=-0.84 upper=0 effort=1000.0 velocity=0.5

Commit message: camera pan and tilt functional and bound

File: src/kenny_description/urdf/kenny.urdf (robot description, URDF)
Before this commit: robot kenny, 9 links, 8 joints
Links:
- removed link camera_tilt
- added link camera_tilt_block; collision box size=${camera_tilt_block_length} ${camera_tilt_block_width} ${ca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; visual box size=${camera_tilt_block_length} ${camera_tilt_block_width} ${ca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
- added link camera_tilt_holder; visual box size=${camera_tilt_holder_length} ${camera_tilt_holder_width} ${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
Joints:
- removed joint camera_tilt_to_pan
- added joint camera_tilt_block_to_holder: type revolute, parent camera_tilt_block, child camera_tilt_holder, origin xyz=0 ${-camera_tilt_holder_length} ${camera_tilt_block_depth/2} rpy=0 0 0, axis 0 1 0, limit lower=${-1*pi/6} upper=${pi/6} effort=1000.0 velocity=0.5
- added joint camera_tilt_block_to_pan: type fixed, parent camera_pan, child camera_tilt_block, origin xyz=0 ${camera_pan_rad} ${camera_pan_rad-camera_tilt_block_width/2} rpy=0 0 0, axis 0 1 0
- joint base_to_reel: origin xyz=${reel_base_offset} 0 ${base_depth+reel_length/2} -> xyz=${reel_base_offset} 0 ${base_depth}
- joint base_to_wheel_left: origin xyz=0 ${-0.5*(base_width+wheel_width)} ${off_floor+(off_floor - wheel_depth)/2} -> xyz=0 ${-0.5*(base_width+wheel_width)} ${-off_floor+wheel_depth/2}
- joint base_to_wheel_right: origin xyz=0 ${0.5*(base_width+wheel_width)} ${off_floor+(off_floor - wheel_depth)/2} -> xyz=0 ${0.5*(base_width+wheel_width)} ${-off_floor+wheel_depth/2}
- joint camera_pan_to_arm1: limit lower=-0.84 upper=0 effort=1000.0 velocity=0.5 -> lower=${-pi/4} upper=${pi/4} effort=1000.0 velocity=0.5

Commit message: splitting urdf for readability

File: src/kenny_description/urdf/kenny.urdf (robot description, URDF)
Before this commit: robot kenny, 10 links, 9 joints
Links:
- removed link arm_link1
- removed link arm_link2
- removed link arm_link3
- removed link base_link
- removed link reel
- removed link wheel_left
- removed link wheel_right
Joints:
- removed joint base_to_reel
- removed joint base_to_wheel_left
- removed joint base_to_wheel_right
- removed joint link1_to_link2
- removed joint link2_to_link3
- removed joint reel_to_link1

Commit message: fixed base collision frame and transform hierarchy

File: src/kenny_description/urdf/kenny.urdf (robot description, URDF)
Before this commit: robot kenny, 0 links, 1 joints
Joints:
- joint arm_mount_joint: origin xyz=${reel_base_offset} 0 ${base_depth+off_floor+0.5*reel_length} -> xyz=${reel_base_offset} 0 ${base_depth/2+0.5*reel_length}
