Commit message: added diffdrive plugin & made wheels round

File: src/kenny_description/urdf/base/base.urdf.xacro (robot description, xacro)
@@ -16,12 +16,14 @@
       <visual>
         <geometry>
-          <box size="${wheel_length} ${wheel_width} ${wheel_depth}"/>
+          <!-- <box size="${wheel_length} ${wheel_width} ${wheel_depth}"/> -->
+            <cylinder length="${wheel_width}" radius="${wheel_depth/2}"/>
         </geometry>
-        <origin xyz="0 0 0"/>
+        <origin xyz="0 0 0" rpy="1.57 0 0"/>
         <material name="black"/>
       </visual>
       <collision>
         <geometry>
-            <box size="${wheel_length} ${wheel_width} ${wheel_depth}"/>
+            <!-- <box size="${wheel_length} ${wheel_width} ${wheel_depth}"/> -->
+            <cylinder length="${wheel_width}" radius="${wheel_depth/2}"/>
         </geometry>
         <!-- <origin xyz="0 0 0"/> -->
@@ -33,10 +35,12 @@
       </inertial>
     </link>
-    <joint name="base_to_${name}" type="fixed">
+    <joint name="joint_base_${name}" type="continuous">
       <parent link="base_link"/>
       <child link="${name}"/>
       <origin xyz="0 ${reflect * 0.5*(base_width+wheel_width)} ${-off_floor+wheel_depth/2}" />
+      <axis xyz="0 1 0"/>
     </joint>
   </xacro:macro>
+  <!--  ++++++++++++++++++++++++++++++++++++++++ -->
   <xacro:macro name="kenny_base" >
     <link name="base_link">

Commit message: created dummy link

File: src/kenny_description/urdf/base/base.urdf.xacro (robot description, xacro)
@@ -66,4 +66,8 @@
       </inertial>
     </link>
+    <joint name="dummy_joint" type="fixed">
+      <parent link="dummy"/>
+      <child link="base_link"/>
+    </joint>
     <xacro:wheel name="wheel_right" reflect="1" />
     <xacro:wheel name="wheel_left" reflect="-1"/>

File: src/kenny_description/urdf/kenny.urdf (robot description, URDF)
Before this commit: robot kenny, 0 links, 0 joints
Links:
- added link dummy

Commit message: drives relative to odom

File: src/kenny_description/urdf/base/base.urdf.xacro (robot description, xacro)
@@ -45,4 +45,5 @@
   <!--  ++++++++++++++++++++++++++++++++++++++++ -->
   <xacro:macro name="kenny_base" >
+    <link name="base_footprint"/>
     <link name="base_link">
       <visual>
@@ -60,4 +61,10 @@
         <origin xyz="0 0 0" />
       </collision>
+    </link>
+    <joint name="base_footprint_joint" type="fixed">
+      <parent link="base_link"/>
+      <child link="base_footprint"/>
+    </joint>
+    <link name="inertial_link">
       <inertial>
         <origin xyz="0 0 ${off_floor+0.5*base_depth}" rpy="0 0 0"/>
@@ -66,7 +73,8 @@
       </inertial>
     </link>
-    <joint name="dummy_joint" type="fixed">
-      <parent link="dummy"/>
-      <child link="base_link"/>
+    <joint name="inertial_joint" type="fixed">
+      <origin xyz="0 0 0" rpy="0 0 0" />
+      <parent link="base_link" />
+      <child link="inertial_link" />
     </joint>
     <xacro:wheel name="wheel_right" reflect="1" />

File: src/kenny_description/urdf/kenny.urdf (robot description, URDF)
Before this commit: robot kenny, 1 links, 0 joints
Links:
- removed link dummy

Commit message: kenny drives

File: src/kenny_description/urdf/base/base.urdf.xacro (robot description, xacro)
@@ -8,8 +8,9 @@
   <xacro:property name="base_width" value="0.444" />
   <xacro:property name="base_depth" value="0.308" />
-  <xacro:property name="off_floor" value="0.05" />
   <xacro:property name="wheel_length" value="1.135" />
   <xacro:property name="wheel_width" value="0.12" />
   <xacro:property name="wheel_depth" value="0.338" />
+  <xacro:property name="wheel_rad" value="0.2" />
+  <xacro:property name="off_floor" value="${wheel_rad - base_depth/2}" />
   <!--  ++++++++++++++++++++++++++++++++++++++++ -->
   <xacro:macro name="wheel" params="name reflect">
@@ -18,5 +19,5 @@
         <geometry>
           <!-- <box size="${wheel_length} ${wheel_width} ${wheel_depth}"/> -->
-            <cylinder length="${wheel_width}" radius="${wheel_depth/2}"/>
+            <cylinder length="${wheel_width}" radius="${wheel_rad}"/>
         </geometry>
         <origin xyz="0 0 0" rpy="1.57 0 0"/>
@@ -26,10 +27,10 @@
         <geometry>
             <!-- <box size="${wheel_length} ${wheel_width} ${wheel_depth}"/> -->
-            <cylinder length="${wheel_width}" radius="${wheel_depth/2}"/>
+            <cylinder length="${wheel_width}" radius="${wheel_rad}"/>
         </geometry>
         <!-- <origin xyz="0 0 0"/> -->
       </collision>
       <inertial>
-        <origin xyz="0 0 ${+0.5*base_depth}" rpy="0 0 0"/>
+        <origin xyz="0 0 ${wheel_rad}" rpy="0 0 0"/>
         <mass value="1"/>
         <inertia ixx="0.2" ixy="0.0" ixz="0.0" iyy="0.2" iyz="0.0" izz="0.2"/>
@@ -39,5 +40,5 @@
       <parent link="base_link"/>
       <child link="${name}"/>
-      <origin xyz="0 ${reflect * 0.5*(base_width+wheel_width)} ${-off_floor+wheel_depth/2}" />
+      <origin xyz="0 ${reflect * 0.5*(base_width+wheel_width)} ${off_floor}" />
       <axis xyz="0 1 0"/>
     </joint>
@@ -78,4 +79,9 @@
       <child link="inertial_link" />
     </joint>
+    <!-- <link name="dummy"></link>
+    <joint name="dummy_joint" type="fixed">
+      <parent link="dummy"/>
+      <child link="inertial_link"/>
+    </joint> -->
     <xacro:wheel name="wheel_right" reflect="1" />
     <xacro:wheel name="wheel_left" reflect="-1"/>

Commit message: changed urdf to have 4 wheels

File: src/kenny_description/urdf/base/base.urdf.xacro (robot description, xacro)
@@ -10,9 +10,9 @@
   <xacro:property name="wheel_length" value="1.135" />
   <xacro:property name="wheel_width" value="0.12" />
-  <xacro:property name="wheel_depth" value="0.338" />
   <xacro:property name="wheel_rad" value="0.2" />
+  <xacro:property name="wheel_sep" value="0.6" />
   <xacro:property name="off_floor" value="${wheel_rad - base_depth/2}" />
   <!--  ++++++++++++++++++++++++++++++++++++++++ -->
-  <xacro:macro name="wheel" params="name reflect">
+  <xacro:macro name="wheel" params="name sidereflect frontback">
     <link name="${name}">
       <visual>
@@ -40,5 +40,5 @@
       <parent link="base_link"/>
       <child link="${name}"/>
-      <origin xyz="0 ${reflect * 0.5*(base_width+wheel_width)} ${off_floor}" />
+      <origin xyz="${frontback * wheel_sep/2} ${sidereflect * 0.5*(base_width+wheel_width)} ${off_floor}" />
       <axis xyz="0 1 0"/>
     </joint>
@@ -84,9 +84,13 @@
       <child link="inertial_link"/>
     </joint> -->
-    <xacro:wheel name="wheel_right" reflect="1" />
-    <xacro:wheel name="wheel_left" reflect="-1"/>
+    <xacro:wheel name="wheel_rfront" sidereflect="1" frontback="1"/>
+    <xacro:wheel name="wheel_rback" sidereflect="1" frontback="-1"/>
+    <xacro:wheel name="wheel_lfront" sidereflect="-1" frontback="1"/>
+    <xacro:wheel name="wheel_lback" sidereflect="-1" frontback="-1"/>
     <!-- Transmission Macros for wheels -->
-    <xacro:kenny_wheel_joint_transmission name="base_wheel_right"/>
-    <xacro:kenny_wheel_joint_transmission name="base_wheel_left"/>
+    <xacro:kenny_wheel_joint_transmission name="base_wheel_rfront"/>
+    <xacro:kenny_wheel_joint_transmission name="base_wheel_rback"/>
+    <xacro:kenny_wheel_joint_transmission name="base_wheel_lfront"/>
+    <xacro:kenny_wheel_joint_transmission name="base_wheel_lback"/>
     <!-- Gazebo Macro -->
     <xacro:base_gazebo/>

Commit message: 4 wheeled Kenny

File: src/kenny_description/urdf/base/base.urdf.xacro (robot description, xacro)
@@ -32,7 +32,7 @@
       </collision>
       <inertial>
-        <origin xyz="0 0 ${wheel_rad}" rpy="0 0 0"/>
+        <origin xyz="0 0 0" rpy="0 0 0"/>
         <mass value="1"/>
-        <inertia ixx="0.2" ixy="0.0" ixz="0.0" iyy="0.2" iyz="0.0" izz="0.2"/>
+        <inertia ixx="0.0" ixy="0.0" ixz="0.0" iyy="0.0" iyz="0.0" izz="0.0"/>
       </inertial>
     </link>

Commit message: kenny can drive now

File: src/kenny_description/urdf/base/base.urdf.xacro (robot description, xacro)
@@ -21,5 +21,5 @@
             <cylinder length="${wheel_width}" radius="${wheel_rad}"/>
         </geometry>
-        <origin xyz="0 0 0" rpy="1.57 0 0"/>
+        <origin xyz="0 0 0" rpy="0 0 0"/>
         <material name="black"/>
       </visual>
@@ -33,6 +33,6 @@
       <inertial>
         <origin xyz="0 0 0" rpy="0 0 0"/>
-        <mass value="1"/>
-        <inertia ixx="0.0" ixy="0.0" ixz="0.0" iyy="0.0" iyz="0.0" izz="0.0"/>
+        <mass value="2"/>
+        <inertia ixx="0.02467" ixy="0.0" ixz="0.0" iyy="0.04411" iyz="0.0" izz="0.02467"/>
       </inertial>
     </link>
@@ -40,6 +40,6 @@
       <parent link="base_link"/>
       <child link="${name}"/>
-      <origin xyz="${frontback * wheel_sep/2} ${sidereflect * 0.5*(base_width+wheel_width)} ${off_floor}" />
-      <axis xyz="0 1 0"/>
+      <origin xyz="${frontback * wheel_sep/2} ${sidereflect * 0.5*(base_width+wheel_width)} ${off_floor}" rpy="1.57 0 0"/>
+      <axis xyz="0 0 1"/>
     </joint>
   </xacro:macro>

Commit message: back to 2 wheeling

File: src/kenny_description/urdf/base/base.urdf.xacro (robot description, xacro)
@@ -11,7 +11,9 @@
   <xacro:property name="wheel_rad" value="0.2" />
   <xacro:property name="wheel_sep" value="0.6" />
-  <xacro:property name="off_floor" value="${wheel_rad - base_depth/2}" />
+  <!-- <xacro:property name="off_floor" value="${wheel_rad - base_depth/2}" /> -->
+  <xacro:property name="off_floor" value="${wheel_rad}" />
   <!--  ++++++++++++++++++++++++++++++++++++++++ -->
-  <xacro:macro name="wheel" params="name sidereflect frontback">
+  <!-- <xacro:macro name="wheel" params="name sidereflect frontback"> -->
+  <xacro:macro name="wheel" params="name reflect">
     <link name="${name}">
       <visual>
@@ -39,5 +41,7 @@
       <parent link="base_link"/>
       <child link="${name}"/>
-      <origin xyz="${frontback * wheel_sep/2} ${sidereflect * 0.5*(base_width+wheel_width)} ${off_floor}" rpy="1.57 0 0"/>
+      <!-- <origin xyz="${frontback * wheel_sep/2} ${sidereflect * 0.5*(base_width+wheel_width)} ${off_floor}" rpy="1.57 0 0"/> -->
+      <!-- <origin xyz="0 ${reflect * 0.5*(base_width+wheel_width)} ${off_floor}" rpy="1.57 0 0"/> -->
+      <origin xyz="0 ${reflect * 0.5*(base_width+wheel_width)} 0" rpy="1.57 0 0"/>
       <axis xyz="0 0 1"/>
     </joint>
@@ -45,5 +49,7 @@
   <!--  ++++++++++++++++++++++++++++++++++++++++ -->
   <xacro:macro name="kenny_base" >
-    <link name="base_footprint"/>
+    <link name="base_footprint">
+      <origin xyz="0 0 0"/>
+    </link>
     <link name="base_link">
       <visual>
@@ -51,5 +57,6 @@
             <box size="${base_length} ${base_width} ${base_depth}"/>
         </geometry>
-        <origin xyz="0 0 ${off_floor+base_depth/2}" />
+        <!-- <origin xyz="0 0 ${off_floor+base_depth/2}" /> -->
+        <origin xyz="0 0 0"/>
         <material name="yellow"/>
       </visual>
@@ -65,4 +72,5 @@
       <parent link="base_link"/>
       <child link="base_footprint"/>
+      <origin xyz="0 0 ${off_floor+base_depth/2}" />
     </joint>
     <link name="inertial_link">
@@ -83,13 +91,20 @@
       <child link="inertial_link"/>
     </joint> -->
-    <xacro:wheel name="wheel_rfront" sidereflect="1" frontback="1"/>
+    <!-- 4 Wheel Kenny -->
+    <xacro:wheel name="wheel_right" reflect="1" />
+    <xacro:wheel name="wheel_left" reflect="-1"/>
+    <xacro:kenny_wheel_joint_transmission name="base_wheel_right"/>
+    <xacro:kenny_wheel_joint_transmission name="base_wheel_left"/>
+    <!-- 4 Wheel Kenny -->
+    <!-- <xacro:wheel name="wheel_rfront" sidereflect="1" frontback="1"/>
     <xacro:wheel name="wheel_rback" sidereflect="1" frontback="-1"/>
     <xacro:wheel name="wheel_lfront" sidereflect="-1" frontback="1"/>
     <xacro:wheel name="wheel_lback" sidereflect="-1" frontback="-1"/>
+     -->
     <!-- Transmission Macros for wheels -->
-    <xacro:kenny_wheel_joint_transmission name="base_wheel_rfront"/>
+    <!-- <xacro:kenny_wheel_joint_transmission name="base_wheel_rfront"/>
     <xacro:kenny_wheel_joint_transmission name="base_wheel_rback"/>
     <xacro:kenny_wheel_joint_transmission name="base_wheel_lfront"/>
-    <xacro:kenny_wheel_joint_transmission name="base_wheel_lback"/>
+    <xacro:kenny_wheel_joint_transmission name="base_wheel_lback"/> -->
     <!-- Gazebo Macro -->
     <xacro:base_gazebo/>

Commit message: drives smoother with caster wheels

File: src/kenny_description/urdf/base/base.urdf.xacro (robot description, xacro)
@@ -11,4 +11,5 @@
   <xacro:property name="wheel_rad" value="0.2" />
   <xacro:property name="wheel_sep" value="0.6" />
+  <xacro:property name="caster_rad" value="${wheel_rad - (base_depth/2)}"/>
   <!-- <xacro:property name="off_floor" value="${wheel_rad - base_depth/2}" /> -->
   <xacro:property name="off_floor" value="${wheel_rad}" />
@@ -47,4 +48,31 @@
     </joint>
   </xacro:macro>
+  <xacro:macro name="caster" params="name reflect">
+    <link name="${name}">
+      <visual>
+        <origin xyz="0 0 0"/>
+        <geometry>
+          <sphere radius="${caster_rad}"/>
+        </geometry>
+      </visual>
+      <collision>
+        <geometry>
+          <sphere radius="${caster_rad}"/>
+        </geometry>
+      </collision>
+      <inertial>
+        <origin xyz="0 0 0" rpy="0 0 0"/>
+        <mass value="0.5"/>
+        <inertia ixx="0.02467" ixy="0.0" ixz="0.0" iyy="0.04411" iyz="0.0" izz="0.02467"/>
+      </inertial>
+    </link>
+    <joint name="joint_base_${name}" type="revolute">
+      <parent link="base_link"/>
+      <child link="${name}"/>
+      <origin xyz="${reflect*(base_length/2-caster_rad)} 0 ${-base_depth/2}"/>
+      <axis xyz="0 0 1"/>
+      <limit effort="1000" lower="0" upper="0" velocity="0"/>
+    </joint>
+  </xacro:macro>
   <!--  ++++++++++++++++++++++++++++++++++++++++ -->
   <xacro:macro name="kenny_base" >
@@ -76,11 +104,11 @@
     <link name="inertial_link">
       <inertial>
-        <origin xyz="0 0 ${off_floor+0.5*base_depth}" rpy="0 0 0"/>
-        <mass value="1"/>
+        <origin xyz="0 0 0" rpy="0 0 0" />
+        <mass value="200"/>
         <inertia ixx="0.2" ixy="0.0" ixz="0.0" iyy="0.2" iyz="0.0" izz="0.2"/>
       </inertial>
     </link>
     <joint name="inertial_joint" type="fixed">
-      <origin xyz="0 0 0" rpy="0 0 0" />
+      <origin xyz="0 0 ${off_floor+0.5*base_depth}" rpy="0 0 0"/>
       <parent link="base_link" />
       <child link="inertial_link" />
@@ -107,4 +135,6 @@
     <xacro:kenny_wheel_joint_transmission name="base_wheel_lfront"/>
     <xacro:kenny_wheel_joint_transmission name="base_wheel_lback"/> -->
+    <xacro:caster name="caster_front" reflect="1"/>
+    <xacro:caster name="caster_back" reflect="-1"/>
     <!-- Gazebo Macro -->
     <xacro:base_gazebo/>
