Commit message: updated parsed urdf

File: src/kenny_description/kennyout.urdf (robot description, URDF)
Before this commit: robot kenny, 12 links, 11 joints
Links:
- removed link wheel_left
- removed link wheel_right
- added link wheel_lback, mass 1; collision cylinder length=0.12 radius=0.2; visual cylinder length=0.12 radius=0.2
- added link wheel_lfront, mass 1; collision cylinder length=0.12 radius=0.2; visual cylinder length=0.12 radius=0.2
- added link wheel_rback, mass 1; collision cylinder length=0.12 radius=0.2; visual cylinder length=0.12 radius=0.2
- added link wheel_rfront, mass 1; collision cylinder length=0.12 radius=0.2; visual cylinder length=0.12 radius=0.2
Joints:
- removed joint joint_base_wheel_left
- removed joint joint_base_wheel_right
- added joint joint_base_wheel_lback: type continuous, parent base_link, child wheel_lback, origin xyz=-0.3 -0.282 0.046, axis 0 1 0
- added joint joint_base_wheel_lfront: type continuous, parent base_link, child wheel_lfront, origin xyz=0.3 -0.282 0.046, axis 0 1 0
- added joint joint_base_wheel_rback: type continuous, parent base_link, child wheel_rback, origin xyz=-0.3 0.282 0.046, axis 0 1 0
- added joint joint_base_wheel_rfront: type continuous, parent base_link, child wheel_rfront, origin xyz=0.3 0.282 0.046, axis 0 1 0
- joint arm_mount_joint: origin xyz=0.0 0 0.403 -> xyz=0.0 0 0.399

Commit message: made all joints gazebo compatible

File: src/kenny_description/kennyout.urdf (robot description, URDF)
Before this commit: robot kenny, 14 links, 13 joints
Links:
- link wheel_lback: mass 1 -> 2
- link wheel_lfront: mass 1 -> 2
- link wheel_rback: mass 1 -> 2
- link wheel_rfront: mass 1 -> 2
Joints:
- joint arm_mount_joint: limit (none) -> lower=0 upper=0 effort=1000.0 velocity=0; type fixed -> revolute
- joint joint_base_wheel_lback: axis 0 1 0 -> 0 0 1; origin xyz=-0.3 -0.282 0.046 -> xyz=-0.3 -0.282 0.046 rpy=1.57 0 0
- joint joint_base_wheel_lfront: axis 0 1 0 -> 0 0 1; origin xyz=0.3 -0.282 0.046 -> xyz=0.3 -0.282 0.046 rpy=1.57 0 0
- joint joint_base_wheel_rback: axis 0 1 0 -> 0 0 1; origin xyz=-0.3 0.282 0.046 -> xyz=-0.3 0.282 0.046 rpy=1.57 0 0
- joint joint_base_wheel_rfront: axis 0 1 0 -> 0 0 1; origin xyz=0.3 0.282 0.046 -> xyz=0.3 0.282 0.046 rpy=1.57 0 0
- joint joint_reel_link1: limit (none) -> lower=-20 upper=20 effort=1000.0 velocity=0; type continuous -> revolute

File: src/kenny_description/urdf/arm/arm.urdf.xacro (robot description, xacro)
@@ -68,10 +68,10 @@
       </inertial>
     </link>
-    <joint name="joint_reel_link1" type="continuous">
+    <joint name="joint_reel_link1" type="revolute">
         <parent link="reel"/>
         <child link="arm_link1"/>
         <origin xyz="${-1*reel_base_offset} 0 ${reel_length/2+link1_depth/2}" rpy="0 0 0"/>
         <axis xyz="0 0 1"/>
-        <!-- <limit effort="1000.0" lower="0" upper="0" velocity="0"/> -->
+        <limit effort="1000.0" lower="-20" upper="20" velocity="0"/>
     </joint>
     <link name="arm_link2">

File: src/kenny_description/urdf/kenny.urdf (robot description, URDF)
Before this commit: robot kenny, 0 links, 1 joints
Joints:
- joint arm_mount_joint: limit (none) -> lower=0 upper=0 effort=1000.0 velocity=0; type fixed -> revolute

Commit message: motorised reel, robot does not spawn in gazebo

File: src/kenny_description/kennyout.urdf (robot description, URDF)
Before this commit: robot kenny, 14 links, 13 joints
Links:
- removed link wheel_lback
- removed link wheel_lfront
- removed link wheel_rback
- removed link wheel_rfront
- added link caster_back, mass 0.5; collision sphere radius=0.046; visual sphere radius=0.046
- added link caster_front, mass 0.5; collision sphere radius=0.046; visual sphere radius=0.046
- added link dummy_reel, mass 1; collision cylinder length=0.09 radius=0.199; visual cylinder length=0.0225 radius=0.199
- added link wheel_left, mass 2; collision cylinder length=0.12 radius=0.2; visual cylinder length=0.12 radius=0.2
- added link wheel_right, mass 2; collision cylinder length=0.12 radius=0.2; visual cylinder length=0.12 radius=0.2
- link inertial_link: mass 1 -> 200
Joints:
- removed joint joint_base_wheel_lback
- removed joint joint_base_wheel_lfront
- removed joint joint_base_wheel_rback
- removed joint joint_base_wheel_rfront
- removed joint joint_link1_link2
- removed joint joint_link2_link3
- removed joint joint_reel_link1
- added joint J0: type revolute, parent dummy_reel, child arm_link1, origin xyz=-0.0 0 0.161 rpy=0 0 0, axis 0 0 1, limit lower=-20 upper=20 effort=1000.0 velocity=0
- added joint J1: type revolute, parent arm_link1, child arm_link2, origin xyz=0.365 0 0 rpy=0 -0.65 0, axis 0 1 0, limit lower=0 upper=1.65 effort=1000.0 velocity=0.5
- added joint J2: type revolute, parent arm_link2, child arm_link3, origin xyz=0 0 0.64 rpy=0 0 0, axis 0 1 0, limit lower=0 upper=0.84 effort=1000.0 velocity=0.5
- added joint J3: type revolute, parent dummy_reel, child reel, axis 0 0 1, limit lower=0 upper=0 effort=1000.0 velocity=0
- added joint dummy_J3: type revolute, parent base_link, child dummy_reel, axis 0 0 0, limit lower=0 upper=0 effort=1000.0 velocity=0
- added joint joint_base_caster_back: type revolute, parent base_link, child caster_back, origin xyz=-0.542 0 -0.154, axis 0 0 1, limit lower=0 upper=0 effort=1000 velocity=0
- added joint joint_base_caster_front: type revolute, parent base_link, child caster_front, origin xyz=0.542 0 -0.154, axis 0 0 1, limit lower=0 upper=0 effort=1000 velocity=0
- added joint joint_base_wheel_left: type continuous, parent base_link, child wheel_left, origin xyz=0 -0.282 0 rpy=1.57 0 0, axis 0 0 1
- added joint joint_base_wheel_right: type continuous, parent base_link, child wheel_right, origin xyz=0 0.282 0 rpy=1.57 0 0, axis 0 0 1
- joint arm_mount_joint: origin xyz=0.0 0 0.399 -> xyz=0.0 0 0.199
- joint base_footprint_joint: origin (none) -> xyz=0 0 0.354
- joint inertial_joint: origin xyz=0 0 0 rpy=0 0 0 -> xyz=0 0 0.354 rpy=0 0 0

File: src/kenny_description/urdf/arm/arm.transmission.xacro (robot description, xacro)
@@ -5,5 +5,5 @@
     <transmission name="tran_${name}">
       <type>transmission_interface/SimpleTransmission</type>
-      <joint name="joint_${name}">
+      <joint name="${name}">
         <hardwareInterface>hardware_interface/PositionJointInterface</hardwareInterface>
       </joint>

File: src/kenny_description/urdf/arm/arm.urdf.xacro (robot description, xacro)
@@ -19,5 +19,30 @@
   <xacro:property name="reel_base_offset" value="0.0" />
   <!--  ++++++++++++++++++++++++++++++++++++++++ -->
-  <xacro:macro name="kenny_arm" > <!-- params="parent *origin"> -->
+  <xacro:macro name="kenny_arm" params="parent"> <!-- params="parent *origin"> -->
+    <link name="dummy_reel">
+      <visual>
+        <geometry>
+          <cylinder length="${reel_length/4}" radius="${reel_rad}"/>
+        </geometry>
+        <origin xyz="0 0 0" rpy="0 0 0"/>
+        <material name="yellow"/>
+      </visual>
+      <collision>
+        <geometry>
+            <cylinder length="${reel_length}" radius="${reel_rad}"/>
+        </geometry>
+      </collision>
+      <inertial>
+        <origin xyz="0 0 0" rpy="0 0 0"/>
+        <mass value="1"/>
+        <inertia ixx="0" ixy="0.0" ixz="0.0" iyy="0.2" iyz="0.0" izz="0"/>
+      </inertial>
+    </link>
+    <joint name="dummy_J3" type="revolute">
+      <parent link="${parent}"/>
+      <child link="dummy_reel"/>
+      <axis xyz="0 0 0"/>
+      <limit effort="1000.0" lower="0" upper="0" velocity="0"/>
+    </joint>
     <link name="reel">
       <visual>
@@ -40,13 +65,12 @@
       </inertial>
     </link>
-    <!-- fixed joints do not exist in gazebo models (SDF file format),
-         fixed joint is now revolute with 0 degrees of motion -->
-    <!-- <joint name="joint_base_reel" type="revolute">
-      <parent link="${parent}"/>
+    <!-- joint between reel and base - allows for motorised reel -->
+    <joint name="J3" type="revolute">
+      <parent link="dummy_reel"/>
       <child link="reel"/>
       <axis xyz="0 0 1"/>
-      <xacro:insert_block name="origin" />
-        <limit effort="1000.0" lower="0" upper="0" velocity="0"/>
-    </joint> -->
+      <!-- <xacro:insert_block name="origin" /> -->
+      <limit effort="1000.0" lower="0" upper="0" velocity="0"/>
+    </joint>
     <link name="arm_link1">
       <visual>
@@ -68,6 +92,7 @@
       </inertial>
     </link>
-    <joint name="joint_reel_link1" type="revolute">
-        <parent link="reel"/>
+    <!-- link between reel and link1 -->
+    <joint name="J0" type="revolute">
+        <parent link="dummy_reel"/>
         <child link="arm_link1"/>
         <origin xyz="${-1*reel_base_offset} 0 ${reel_length/2+link1_depth/2}" rpy="0 0 0"/>
@@ -95,5 +120,6 @@
       </inertial>
     </link>
-    <joint name="joint_link1_link2" type="revolute">
+    <!-- joint between link1 and link2 -->
+    <joint name="J1" type="revolute">
       <parent link="arm_link1"/>
       <child link="arm_link2"/>
@@ -123,5 +149,6 @@
       </inertial>
     </link>
-    <joint name="joint_link2_link3" type="revolute">
+  <!-- joint between link 2 and link 3 -->
+    <joint name="J2" type="revolute">
       <parent link="arm_link2"/>
       <child link="arm_link3"/>
@@ -131,7 +158,8 @@
     </joint>
     <!-- Transmission Macros -->
-    <xacro:kenny_arm_joint_transmission name="reel_link1"/>
-    <xacro:kenny_arm_joint_transmission name="link1_link2"/>
-    <xacro:kenny_arm_joint_transmission name="link2_link3"/>
+    <xacro:kenny_arm_joint_transmission name="J0"/>
+    <xacro:kenny_arm_joint_transmission name="J1"/>
+    <xacro:kenny_arm_joint_transmission name="J2"/>
+    <xacro:kenny_arm_joint_transmission name="J3"/>
     <!-- Gazebo Macro -->
     <xacro:kenny_arm_gazebo/>

Commit message: changed arm joint names

File: src/kenny_description/kennyout.urdf (robot description, URDF)
Before this commit: robot kenny, 15 links, 15 joints
Links:
- removed link arm_link1
- removed link arm_link2
- removed link arm_link3
- added link arm, mass 1; collision box size=0.73 0.378 0.232; visual box size=0.73 0.378 0.232
- added link forearm, mass 1; collision box size=0.18 0.389 0.64; visual box size=0.18 0.389 0.64
- added link hand, mass 1; collision box size=0.788 0.06 0.08; visual box size=0.788 0.06 0.08
Joints:
- removed joint J0
- removed joint J1
- removed joint J2
- removed joint J3
- removed joint dummy_J3
- added joint dummy_reel_joint: type revolute, parent base_link, child dummy_reel, axis 0 0 0, limit lower=0 upper=0 effort=1000.0 velocity=0
- added joint elbow: type revolute, parent arm, child forearm, origin xyz=0.365 0 0 rpy=0 -0.65 0, axis 0 1 0, limit lower=0 upper=1.65 effort=1000.0 velocity=0.5
- added joint reel_joint: type revolute, parent dummy_reel, child reel, axis 0 0 1, limit lower=0 upper=0 effort=1000.0 velocity=0
- added joint shoulder: type revolute, parent dummy_reel, child arm, origin xyz=-0.0 0 0.161 rpy=0 0 0, axis 0 0 1, limit lower=-20 upper=20 effort=1000.0 velocity=0
- added joint wrist: type revolute, parent forearm, child hand, origin xyz=0 0 0.64 rpy=0 0 0, axis 0 1 0, limit lower=0 upper=0.84 effort=1000.0 velocity=0.5
- joint joint_camera_z_rotation: parent arm_link1 -> arm

File: src/kenny_description/urdf/arm/arm.urdf.xacro (robot description, xacro)
@@ -5,14 +5,14 @@
   <xacro:include filename="$(find kenny_description)/urdf/arm/arm.gazebo.urdf"/>
   <!--  ++++++++++++++++++++++++++++++++++++++++ -->
-  <xacro:property name="link1_length" value="0.73"/>
-  <xacro:property name="link1_width" value="0.378"/>
-  <xacro:property name="link1_depth" value="0.232"/>
-  <xacro:property name="link2_length" value="0.64"/>
-  <xacro:property name="link2_width" value="0.389"/>
-  <xacro:property name="link2_depth" value="0.18"/>
-  <xacro:property name="link2_default_rotation" value="-0.65"/>
-  <xacro:property name="link3_length" value="0.788"/>
-  <xacro:property name="link3_width" value="0.06"/>
-  <xacro:property name="link3_depth" value="0.08"/>
+  <xacro:property name="arm_length" value="0.73"/>
+  <xacro:property name="arm_width" value="0.378"/>
+  <xacro:property name="arm_depth" value="0.232"/>
+  <xacro:property name="forearm_length" value="0.64"/>
+  <xacro:property name="forearm_width" value="0.389"/>
+  <xacro:property name="forearm_depth" value="0.18"/>
+  <xacro:property name="forearm_default_rotation" value="-0.65"/>
+  <xacro:property name="hand_length" value="0.788"/>
+  <xacro:property name="hand_width" value="0.06"/>
+  <xacro:property name="hand_depth" value="0.08"/>
   <xacro:property name="reel_rad" value="0.199" />
   <xacro:property name="reel_length" value="0.09" />
@@ -39,5 +39,5 @@
       </inertial>
     </link>
-    <joint name="dummy_J3" type="revolute">
+    <joint name="dummy_reel_joint" type="revolute">
       <parent link="${parent}"/>
       <child link="dummy_reel"/>
@@ -66,5 +66,5 @@
     </link>
     <!-- joint between reel and base - allows for motorised reel -->
-    <joint name="J3" type="revolute">
+    <joint name="reel_joint" type="revolute">
       <parent link="dummy_reel"/>
       <child link="reel"/>
@@ -73,8 +73,8 @@
       <limit effort="1000.0" lower="0" upper="0" velocity="0"/>
     </joint>
-    <link name="arm_link1">
+    <link name="arm">
       <visual>
         <geometry>
-          <box size="${link1_length} ${link1_width} ${link1_depth}"/>
+          <box size="${arm_length} ${arm_width} ${arm_depth}"/>
         </geometry>
         <material name="yellow"/>
@@ -83,5 +83,5 @@
       <collision>
         <geometry>
-          <box size="${link1_length} ${link1_width} ${link1_depth}"/>
+          <box size="${arm_length} ${arm_width} ${arm_depth}"/>
         </geometry>
       </collision>
@@ -92,25 +92,25 @@
       </inertial>
     </link>
-    <!-- link between reel and link1 -->
-    <joint name="J0" type="revolute">
+    <!-- link between reel and arm -->
+    <joint name="shoulder" type="revolute">
         <parent link="dummy_reel"/>
-        <child link="arm_link1"/>
-        <origin xyz="${-1*reel_base_offset} 0 ${reel_length/2+link1_depth/2}" rpy="0 0 0"/>
+        <child link="arm"/>
+        <origin xyz="${-1*reel_base_offset} 0 ${reel_length/2+arm_depth/2}" rpy="0 0 0"/>
         <axis xyz="0 0 1"/>
         <limit effort="1000.0" lower="-20" upper="20" velocity="0"/>
     </joint>
-    <link name="arm_link2">
+    <link name="forearm">
       <visual>
         <geometry>
-            <box size="${link2_depth} ${link2_width} ${link2_length}"/>
+            <box size="${forearm_depth} ${forearm_width} ${forearm_length}"/>
         </geometry>
-        <origin xyz="0 0 ${link2_length/2}" rpy="0 0 0"/>
+        <origin xyz="0 0 ${forearm_length/2}" rpy="0 0 0"/>
         <material name="yellow"/>
       </visual>
       <collision>
         <geometry>
-            <box size="${link2_depth} ${link2_width} ${link2_length}"/>
+            <box size="${forearm_depth} ${forearm_width} ${forearm_length}"/>
         </geometry>
-        <origin xyz="0 0 ${link2_length/2}" rpy="0 0 0"/>
+        <origin xyz="0 0 ${forearm_length/2}" rpy="0 0 0"/>
       </collision>
       <inertial>
@@ -120,26 +120,26 @@
       </inertial>
     </link>
-    <!-- joint between link1 and link2 -->
-    <joint name="J1" type="revolute">
-      <parent link="arm_link1"/>
-      <child link="arm_link2"/>
+    <!-- joint between arm and forearm -->
+    <joint name="elbow" type="revolute">
+      <parent link="arm"/>
+      <child link="forearm"/>
       <axis xyz="0 1 0"/>
-      <origin xyz="${link1_length/2} 0 0" rpy="0 ${link2_default_rotation} 0"/>
-      <!-- <origin xyz="${link1_length/2-link2_depth/2} 0 0" rpy="0 0 0"/> -->
+      <origin xyz="${arm_length/2} 0 0" rpy="0 ${forearm_default_rotation} 0"/>
+      <!-- <origin xyz="${arm_length/2-forearm_depth/2} 0 0" rpy="0 0 0"/> -->
       <limit effort="1000.0" lower="0" upper="1.65" velocity="0.5"/>
     </joint>
-    <link name="arm_link3">
+    <link name="hand">
       <visual>
         <geometry>
-          <box size="${link3_length} ${link3_width} ${link3_depth}"/>
+          <box size="${hand_length} ${hand_width} ${hand_depth}"/>
         </geometry>
-        <origin xyz="${link3_length/2} 0 0" rpy="0 0 0"/>
+        <origin xyz="${hand_length/2} 0 0" rpy="0 0 0"/>
         <material name="yellow"/>
       </visual>
       <collision>
         <geometry>
-          <box size="${link3_length} ${link3_width} ${link3_depth}"/>
+          <box size="${hand_length} ${hand_width} ${hand_depth}"/>
         </geometry>
-        <origin xyz="${link3_length/2} 0 0" rpy="0 0 0"/>
+        <origin xyz="${hand_length/2} 0 0" rpy="0 0 0"/>
       </collision>
       <inertial>
@@ -149,17 +149,17 @@
       </inertial>
     </link>
-  <!-- joint between link 2 and link 3 -->
-    <joint name="J2" type="revolute">
-      <parent link="arm_link2"/>
-      <child link="arm_link3"/>
+  <!-- joint between forearm and hand -->
+    <joint name="wrist" type="revolute">
+      <parent link="forearm"/>
+      <child link="hand"/>
       <axis xyz="0 1 0"/>
-      <origin xyz="0 0 ${link2_length}" rpy="0 0 0"/>
+      <origin xyz="0 0 ${forearm_length}" rpy="0 0 0"/>
       <limit effort="1000.0" lower="0" upper="0.84" velocity="0.5"/>
     </joint>
     <!-- Transmission Macros -->
-    <xacro:kenny_arm_joint_transmission name="J0"/>
-    <xacro:kenny_arm_joint_transmission name="J1"/>
-    <xacro:kenny_arm_joint_transmission name="J2"/>
-    <xacro:kenny_arm_joint_transmission name="J3"/>
+    <xacro:kenny_arm_joint_transmission name="shoulder"/>
+    <xacro:kenny_arm_joint_transmission name="elbow"/>
+    <xacro:kenny_arm_joint_transmission name="wrist"/>
+    <xacro:kenny_arm_joint_transmission name="reel_joint"/>
     <!-- Gazebo Macro -->
     <xacro:kenny_arm_gazebo/>

File: src/kenny_description/urdf/camera_mechanism/camera_mechanism.urdf.xacro (robot description, xacro)
@@ -34,9 +34,9 @@
     </link>
     <joint name="joint_camera_z_rotation" type="revolute">
-      <!-- <parent link="arm_link1"/> -->
+      <!-- <parent link="arm"/> -->
       <parent link="${parent}"/>
       <child link="camera_pan"/>
       <axis xyz="0 0 1"/>
-      <!-- <origin xyz="${pan_arm_offset} 0 ${link1_depth/2}" rpy="0 0 0"/> -->
+      <!-- <origin xyz="${pan_arm_offset} 0 ${arm_depth/2}" rpy="0 0 0"/> -->
       <xacro:insert_block name="origin"/>
       <limit effort="1000.0" lower="${-pi/4}" upper="${pi/4}" velocity="0.5"/>
